File: 02.Hardware/MK1-RP2040/04.TEST-PLUG/Test-plug.brd (EAGLE design)
At the start: 76 x 24 mm, 3 parts, among them J1 PJRAN1X1U01X

Commit message: PCB Test plug v1
Parts:
- moved REPOT_2 7.00 mm to (63.0, 28.0)
- moved J1 2.00 mm to (6.00, 23.0)
Routing:
- net VCC: track 73.7 -> 143.2 mm
- net GND: track 17.1 -> 18.8 mm
Other:
- board size 76 x 24 mm -> 83 x 20 mm
- board text added: "USE ONLY TEST MODE 1 min MAX"
- board text removed: "Use only Test Mode 1 min MAX"
