File: 02.Hardware/MK1-RP2040/04.TEST-PLUG/Test-plug.sch (EAGLE design)
At the start: 3 parts, among them J1 PJRAN1X1U01X

Commit message: PCB Test plug v1
Other:
- moved on the sheet: J1
Changed lines of the file:
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@@
 </classes>
 <parts>
-<part name="J1" library="Connectors" library_urn="urn:adsk.eagle:library:14555660" deviceset="PJRAN1X1U01X" device="" package3d_urn="urn:adsk.eagle:package:10989925/2"/>
+<part name="J1" library="Connectors" deviceset="PJRAN1X1U01X" device="" package3d_urn="urn:adsk.eagle:package:10989925/2"/>
 <part name="RPOT_1" library="BeagleBone_Blue_R3" library_urn="urn:adsk.eagle:library:5828899" deviceset="TESTPAD/W_HOLE_1X1" device="" package3d_urn="urn:adsk.eagle:package:5829473/2"/>
 <part name="REPOT_2" library="BeagleBone_Blue_R3" library_urn="urn:adsk.eagle:library:5828899" deviceset="TESTPAD/W_HOLE_1X1" device="" package3d_urn="urn:adsk.eagle:package:5829473/2"/>
@@
 </plain>
 <instances>
-<instance part="J1" gate="G$1" x="34.29" y="60.96" smashed="yes">
-<attribute name="NAME" x="27.9391" y="66.04071875" size="1.77825" layer="95"/>
-<attribute name="VALUE" x="27.930740625" y="54.600740625" size="1.780590625" layer="96"/>
+<instance part="J1" gate="G$1" x="31.75" y="60.96" smashed="yes">
+<attribute name="NAME" x="25.3991" y="66.04071875" size="1.77825" layer="95"/>
+<attribute name="VALUE" x="25.390740625" y="54.600740625" size="1.780590625" layer="96"/>
 </instance>
 <instance part="RPOT_1" gate="G$1" x="78.74" y="68.58" smashed="yes" rot="R90">
@@
 <segment>
 <pinref part="J1" gate="G$1" pin="2"/>
-<wire x1="39.37" y1="63.5" x2="48.26" y2="63.5" width="0.1524" layer="91"/>
+<wire x1="36.83" y1="63.5" x2="48.26" y2="63.5" width="0.1524" layer="91"/>
 <label x="53.34" y="63.5" size="1.778" layer="95"/>
 <pinref part="J1" gate="G$1" pin="3"/>
 <wire x1="48.26" y1="63.5" x2="78.74" y2="63.5" width="0.1524" layer="91"/>
-<wire x1="39.37" y1="60.96" x2="48.26" y2="60.96" width="0.1524" layer="91"/>
+<wire x1="36.83" y1="60.96" x2="48.26" y2="60.96" width="0.1524" layer="91"/>
 <wire x1="48.26" y1="60.96" x2="48.26" y2="63.5" width="0.1524" layer="91"/>
 <junction x="48.26" y="63.5"/>
@@
 <segment>
 <pinref part="J1" gate="G$1" pin="1"/>
-<wire x1="39.37" y1="58.42" x2="78.74" y2="58.42" width="0.1524" layer="91"/>
+<wire x1="36.83" y1="58.42" x2="78.74" y2="58.42" width="0.1524" layer="91"/>
 <label x="53.34" y="58.42" size="1.778" layer="95"/>
 <pinref part="REPOT_2" gate="G$1" pin="TP"/>
