File: 02.Hardware/MK1-RP2040 - USBC/01.EDCPSU/EDCPSUMK1-RP2040-USBC.brd (EAGLE design)
At the start: 96 x 60.8 mm, 209 parts, among them J1 DX07S016JA1R1500, J6 Display, Q2 2N7002PW, Q4 2N7002PW, Q5 2N7002PW, Q9 2N7002PW, U1 RP2040TR7, U10 IP2721, U11 AP63203, U12 AP64501SP-13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

Commit message: Version 1 para Seti Mk1 USBC Rp2040
Parts:
- R19: value 1K -> 1k
Routing:
- net SAFETY_EN_DCDC: track 55.8 -> 58.9 mm
- net VOUT: track 50.0 -> 48.1 mm
- net N$16: track 46.4 -> 45.3 mm
- net IN+: track 33.9 -> 33.2 mm
- net GND: track 231.1 -> 231.7 mm
- net SCL: track 87.1 -> 86.6 mm
Other:
- board text added: "MK1-RP2040 v1-Jul-2025"
- board text removed: "MK2-RP2040 v2-May-2023"
