File: 02.Hardware/MK1-RP2040 - USBC/01.EDCPSU/EDCPSUMK1-RP2040-USBC.sch (EAGLE design)
At the start: 209 parts, among them J1 DX07S016JA1R1500, J6 Display, Q2 2N7002PW, Q4 2N7002PW, Q5 2N7002PW, Q9 2N7002PW, U1 RP2040TR7, U10 IP2721, U11 AP63203, U12 AP64501SP-13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

Commit message: Version 1 para Seti Mk1 USBC Rp2040
Parts:
- R19: value 1K -> 1k
Other:
- note removed: "Linea de corte en PCB"
- moved on the sheet: RSENSE
